File: pcb/keybowl_core_pcb/keybowl_core_pcb.kicad_pcb (KiCad board)
At the start: 2 copper layers, 174.1 x 118 mm, 38 parts, among them J1 e-Paper Module, J2 e-Paper Module, J3 R200 UHF RFID module, J4 USB_C_Receptacle, SW1 SW_Push, SW2 SW_Push, SW3 SW_Push, SW4 SW_Push, SW5 SW_Push, SW6 SW_Push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

Commit message: working on pcb
Routing:
- net COL2: track 144.1 -> 141.8 mm
- net GPIO18: track 68.7 -> 67.5 mm
Other:
- outline, holes or cut-outs redrawn
- board text added: "... you only need one the other is just for good measure"
- board text added: "4.2{dblquote} ePaper mounting"
- board text added: "Another one here ..."
- board text added: "Nooo not this side pinheaders or similar go on the back"
- board text added: "Oh a big hole don't fall into that"
- board text added: "Oh a via never seen one before :)"
- board text added: "Please turn the PCB and put the Raspberry Pi on the other side."
- board text added: "Put one switch here ..."
- board text added: "Put pinheaders ot similar here"
- board text added: "Some cool Neopixels"
- board text added: "Switches on this side too ..."
- board text added: "The backside ..."
- board text added: "USB C port from the back"
- board text added: "WS2812B LEDs did you see that rainbow?"
- board text added: "Waveshare here"
- board text added: "WeAct Studio here"
- board text added: "You got the idea ..."
- board text added: "a USB C port for supplying power nice!"
- board text added: "a diode"
- board text added: "a small little levelshifter"
- board text added: "a via"
- board text added: "ePaper cable hole"
- board text added: "here connect the RFID module"
- board text added: "here your Raspberry ..."
- board text added: "keyswitch from the back solder here"
- board text added: "more diods"
- board text added: "more holes if you want to mount your RPi"
- board text added: "more switches from the backside"
- board text added: "put your keys inside the bowl"
- board text added: "some capacitors"
- board text added: "some holes"
