File: pcb/keybowl_core_pcb/keybowl_core_pcb.kicad_sch (KiCad schematic)
At the start: 38 parts, among them J1 e-Paper Module, J2 e-Paper Module, J3 R200 UHF RFID module, J4 USB_C_Receptacle, SW1 SW_Push, SW2 SW_Push, SW3 SW_Push, SW4 SW_Push, SW5 SW_Push, SW6 SW_Push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

Commit message: adding firmware and fix small issue inside schematic
Connections:
- net GPIO18 renamed GPIO16
Changed lines of the file:
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@@
 		)
 	)
-	(global_label "GPIO18"
+	(global_label "GPIO16"
 		(shape input)
 		(at 29.21 96.52 180)
@@
 		)
 	)
-	(global_label "GPIO18"
+	(global_label "GPIO16"
 		(shape input)
 		(at 200.66 92.71 0)

Commit message: small chnages on the pcb and extend BOM to PCB assembly parts
Parts:
- C10: value 1000uF -> 10uF
Changed lines of the file:
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@@
 			)
 		)
-		(property "Value" "1000uF"
+		(property "Value" "10uF"
 			(at 33.02 45.7199 0)
 			(effects
